File: VFD Replacement/VFD Replacement.kicad_pcb (KiCad board)
At the start: 2 copper layers, 65 x 27.5 mm, 45 parts, among them J1 Conn_01x05_Pin, J2 Conn_01x05_Pin, J3 Conn_01x06_Pin, J4 Conn_01x06_Pin, J5 Conn_01x02_Pin, Q1 MMDT2222A, Q10 MMDT2222A, Q2 MMDT2222A, Q3 MMDT2222A, Q4 MMDT2222A, Q5 MMDT2222A, Q6 MMDT2222A, Q7 MMDT2222A, Q8 MMDT2222A, Q9 MMDT2222A

Commit message: Update values from sim
Parts:
- R1, R2, R3, R4, R5, R6, R7, R8: value 2.4k -> 12k
- R25: value 10k -> 12k
- R26, R27, R28, R29, R30, R31, R32, R33, R34, R35, R36, R37: value 12k -> 56k
Changed lines of the file:
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@@
       (effects (font (size 1 1) (thickness 0.15)))
     )
-    (property "Value" "12k" (at 0 1.43 0) (layer "F.Fab")
+    (property "Value" "56k" (at 0 1.43 0) (layer "F.Fab")
       (effects (font (size 1 1) (thickness 0.15)))
     )
@@
       (effects (font (size 1 1) (thickness 0.15)))
     )
-    (property "Value" "2.4k" (at 0 1.43 -90) (layer "F.Fab")
+    (property "Value" "12k" (at 0 1.43 -90) (layer "F.Fab")
       (effects (font (size 1 1) (thickness 0.15)))
     )
@@
       (effects (font (size 1 1) (thickness 0.15)))
     )
-    (property "Value" "12k" (at 0 1.43 180) (layer "F.Fab")
+    (property "Value" "56k" (at 0 1.43 180) (layer "F.Fab")
       (effects (font (size 1 1) (thickness 0.15)))
     )
@@
       (effects (font (size 1 1) (thickness 0.15)))
     )
-    (property "Value" "12k" (at 0 1.43 180) (layer "F.Fab")
+    (property "Value" "56k" (at 0 1.43 180) (layer "F.Fab")
       (effects (font (size 1 1) (thickness 0.15)))
     )
@@
       (effects (font (size 1 1) (thickness 0.15)))
     )
-    (property "Value" "2.4k" (at 0.05 0.73 90) (layer "F.Fab")
+    (property "Value" "12k" (at 0.05 0.73 90) (layer "F.Fab")
       (effects (font (size 1 1) (thickness 0.15)))
     )
@@
       (effects (font (size 1 1) (thickness 0.15)))
     )
-    (property "Value" "12k" (at 0 1.43 180) (layer "F.Fab")
+    (property "Value" "56k" (at 0 1.43 180) (layer "F.Fab")
       (effects (font (size 1 1) (thickness 0.15)))
     )
@@
       (effects (font (size 1 1) (thickness 0.15)))
     )
-    (property "Value" "2.4k" (at -0.0125 1.43 90) (layer "F.Fab")
+    (property "Value" "12k" (at -0.0125 1.43 90) (layer "F.Fab")
       (effects (font (size 1 1) (thickness 0.15)))
     )
@@
       (effects (font (size 1 1) (thickness 0.15)))
     )
-    (property "Value" "12k" (at 0 1.43 0) (layer "F.Fab")
+    (property "Value" "56k" (at 0 1.43 0) (layer "F.Fab")
       (effects (font (size 1 1) (thickness 0.15)))
     )
@@
       (effects (font (size 1 1) (thickness 0.15)))
     )
-    (property "Value" "12k" (at 0 1.43 180) (layer "F.Fab")
+    (property "Value" "56k" (at 0 1.43 180) (layer "F.Fab")
       (effects (font (size 1 1) (thickness 0.15)))
     )
@@
       (effects (font (size 1 1) (thickness 0.15)))
     )
-    (property "Value" "12k" (at 0 1.43 0) (layer "F.Fab")
+    (property "Value" "56k" (at 0 1.43 0) (layer "F.Fab")
       (effects (font (size 1 1) (thickness 0.15)))
     )
@@
       (effects (font (size 1 1) (thickness 0.15)))
     )
-    (property "Value" "12k" (at 0 1.43 0) (layer "F.Fab")
+    (property "Value" "56k" (at 0 1.43 0) (layer "F.Fab")
       (effects (font (size 1 1) (thickness 0.15)))
     )
@@
       (effects (font (size 1 1) (thickness 0.15)))
     )
-    (property "Value" "2.4k" (at 0 1.43 90) (layer "F.Fab")
+    (property "Value" "12k" (at 0 1.43 90) (layer "F.Fab")
       (effects (font (size 1 1) (thickness 0.15)))
     )
@@
       (effects (font (size 1 1) (thickness 0.15)))
     )
-    (property "Value" "12k" (at 0 1.43 0) (layer "F.Fab")
+    (property "Value" "56k" (at 0 1.43 0) (layer "F.Fab")
       (effects (font (size 1 1) (thickness 0.15)))
     )
@@
       (effects (font (size 1 1) (thickness 0.15)))
     )
-    (property "Value" "10k" (at 0 1.43 180) (layer "F.Fab")
+    (property "Value" "12k" (at 0 1.43 180) (layer "F.Fab")
       (effects (font (size 1 1) (thickness 0.15)))
     )
@@
       (effects (font (size 1 1) (thickness 0.15)))
     )
-    (property "Value" "2.4k" (at 0 1.43 90) (layer "F.Fab")
+    (property "Value" "12k" (at 0 1.43 90) (layer "F.Fab")
       (effects (font (size 1 1) (thickness 0.15)))
     )
@@
       (effects (font (size 1 1) (thickness 0.15)))
     )
-    (property "Value" "12k" (at 0 1.43 0) (layer "F.Fab")
+    (property "Value" "56k" (at 0 1.43 0) (layer "F.Fab")
       (effects (font (size 1 1) (thickness 0.15)))
     )
@@
       (effects (font (size 1 1) (thickness 0.15)))
     )
-    (property "Value" "2.4k" (at 0 1.43 90) (layer "F.Fab")
+    (property "Value" "12k" (at 0 1.43 90) (layer "F.Fab")
       (effects (font (size 1 1) (thickness 0.15)))
     )
@@
       (effects (font (size 1 1) (thickness 0.15)))
     )
-    (property "Value" "12k" (at 0 1.43 180) (layer "F.Fab")
+    (property "Value" "56k" (at 0 1.43 180) (layer "F.Fab")
       (effects (font (size 1 1) (thickness 0.15)))
     )
@@
       (effects (font (size 1 1) (thickness 0.15)))
     )
-    (property "Value" "2.4k" (at 0 1.43 90) (layer "F.Fab")
+    (property "Value" "12k" (at 0 1.43 90) (layer "F.Fab")
       (effects (font (size 1 1) (thickness 0.15)))
     )
@@
       (effects (font (size 1 1) (thickness 0.15)))
     )
-    (property "Value" "2.4k" (at 0 1.43 90) (layer "F.Fab")
+    (property "Value" "12k" (at 0 1.43 90) (layer "F.Fab")
       (effects (font (size 1 1) (thickness 0.15)))
     )
@@
       (effects (font (size 1 1) (thickness 0.15)))
     )
-    (property "Value" "12k" (at 0 1.43 180) (layer "F.Fab")
-      (effects (font (size 1 1) (thickness 0.15)))
-    )
+    (property "Value" "56k" (at 0 1.43 180) (layer "F.Fab")
+      (effects (font (size 1 1) (thickness 0.15)))
+    )
